Commit message: changed example robot to red

File: example_robot/example_robot_description/urdf/example_robot.urdf.xacro (robot description, xacro)
@@ -15,5 +15,5 @@
   <material name="dark_grey"><color rgba="0.2 0.2 0.2 1.0" /></material>
   <material name="light_grey"><color rgba="0.4 0.4 0.4 1.0" /></material>
-  <material name="yellow"><color rgba="0.8 0.8 0.0 1.0" /></material>
+  <material name="red"><color rgba="0.8 0 0.0 1.0" /></material>
   <material name="black"><color rgba="0.15 0.15 0.15 1.0" /></material>
   <xacro:macro name="wheel" params="prefix *joint_pose">
@@ -117,5 +117,5 @@
           <mesh filename="package://example_robot_description/meshes/jackal-fender.stl"/>
         </geometry>
-        <material name="yellow" />
+        <material name="red" />
       </visual>
     </link>
@@ -127,5 +127,5 @@
           <mesh filename="package://example_robot_description/meshes/accessory_fender.stl"/>
         </geometry>
-        <material name="yellow" />
+        <material name="red" />
       </visual>
     </link>
@@ -148,5 +148,5 @@
           <mesh filename="package://example_robot_description/meshes/jackal-fender.stl"/>
         </geometry>
-        <material name="yellow" />
+        <material name="red" />
       </visual>
     </link>
@@ -158,5 +158,5 @@
           <mesh filename="package://example_robot_description/meshes/accessory_fender.stl"/>
         </geometry>
-        <material name="yellow" />
+        <material name="red" />
       </visual>
     </link>
@@ -222,5 +222,5 @@
   </joint>
   <!-- Bring in simulation data for Gazebo. -->
-  <xacro:include filename="$(find example_robot_description)/urdf/jackal.gazebo" />
+  <xacro:include filename="$(find example_robot_description)/urdf/example_robot.gazebo" />
   <!-- Optional standard accessories, including their simulation data. The rendering
        of these into the final description is controlled by optenv variables, which
